File: sheet_2.kicad_sch (KiCad schematic)
At the start: 4 parts, among them J5 Conn_01x09_Pin, J6 Conn_01x04_Pin, J7 Conn_02x03_Odd_Even, J8 Conn_01x04_Pin

Commit message: done with schematic
Parts:
- J1: renamed from J6; Purpose (none) -> I2C
- J2: renamed from J5; Purpose (none) -> GPIO
- J3: renamed from J8; Purpose (none) -> serial
- J4: renamed from J7; Purpose (none) -> ICSP
Connections:
- net D2: now reaches J2.1 (Pin_1)
- net D3: now reaches J2.2 (Pin_2)
- net D4: now reaches J2.3 (Pin_3)
- net D5: now reaches J2.4 (Pin_4)
- net D6: now reaches J2.5 (Pin_5)
- net D7: now reaches J2.6 (Pin_6)
- net D8: now reaches J2.7 (Pin_7)
- net GND: now reaches J2.8 (Pin_8)
- net GND: now also J1.1 (Pin_1), J3.1 (Pin_1), J4.6 (Pin_6)
- net Vcc: now reaches J2.9 (Pin_9)
- net Vcc: now also J1.2 (Pin_2), J3.2 (Pin_2), J4.2 (Pin_2)
- net SDA: now reaches J1.3 (Pin_3)
- net SCK: now reaches J1.4 (Pin_4)
- net SCK: now also J4.3 (Pin_3)
- net MISO: now reaches J4.1 (Pin_1)
- net MOSI: now reaches J4.4 (Pin_4)
- net RESET: now reaches J4.5 (Pin_5)
- net RX: now reaches J3.3 (Pin_3)
- net TX: now reaches J3.4 (Pin_4)
Other:
- title: mcu_data_logger -> $(project_name)
- moved on the sheet: J1, J3, J4

Commit message: assigned GND and /Vcc to the power net class
Other:
- title: $(project_name) -> ${project_name}
Changed lines of the file:
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@@
 	(paper "A4")
 	(title_block
-		(title "$(project_name)")
+		(title "${project_name}")
 		(rev "1")
 		(company "electron")
